File: ui_submodule.kicad_sch (KiCad schematic)
At the start: 0 parts

Commit message: Finished Squematics V1
Parts:
- added C10, C11: 4.7uF, symbol Device:C_US
- added C9: 4.7k, symbol Device:C_US
- added D2: RED, symbol Device:LED
- added D3: GREEN, symbol Device:LED
- added D4: BLUE, symbol Device:LED
- added J2: Barrel_Jack_MountingPin, symbol Connector:Barrel_Jack_MountingPin
- added R18, R19: 220, symbol Device:R
- added R20: 100, symbol Device:R
- added R21, R22, R23: 1k, symbol Device:R
- added R24, R25, R26: 2.7k, symbol Device:R
- added R27, R28, R29: 3.3k, symbol Device:R
- added RV1: R_Potentiometer, symbol Device:R_Potentiometer
- added SW1: Right, symbol Switch:SW_Omron_B3FS
- added SW2: Left, symbol Switch:SW_Omron_B3FS
- added SW3: SW_SPST, symbol Switch:SW_SPST
- added SW4: Stop, symbol Switch:SW_Omron_B3FS
- added U3: 20x4 LCD, Display:NHD-0420H1Z, symbol Display_Character:NHD-0420H1Z
- added U4: 74LS14, symbol 74xx:74LS14
Connections:
- new net: R25.2, R28.1, SW2.2
- new net: C10.1, R28.2, U4.3
- new net: C9.1, R27.2, U4.1
- new net: C11.1, R29.2, U4.5
- new net: RV1.2, U3.3 (VO)
- new net: R26.2, R29.1, SW4.2
- new net: R24.2, R27.1, SW1.2
- new net: R22.1, U4.11
- new net: D2.2 (A), R18.1
- new net: R21.1, U4.9
- new net: D4.2 (A), R20.1
- new net: J2.1, SW3.1 (A)
- new net: D3.2 (A), R19.1
- new net: R23.1, U4.13
- new net +3.3V: R24.1, R25.1, R26.1
- new net +5V: SW3.2 (B), U3.15 (A), U3.2 (VDD), U4.14 (VCC)
- new net GND: C10.2, C11.2, C9.2, D2.1 (K), D3.1 (K), D4.1 (K), J2.2, R21.2, R22.2, R23.2, RV1.1, SW1.1, SW2.1, SW4.1, U3.1 (VSS), U3.16 (K), U3.5 (R/W), U4.7 (GND)
- new net HALTED: R18.2
- new net LCD_D4: U3.11 (DB4)
- new net LCD_D5: U3.12 (DB5)
- new net LCD_D6: U3.13 (DB6)
- new net LCD_D7: U3.14 (DB7)
- new net LCD_E: U3.6 (E)
- new net LCD_RS: U3.4 (RS)
- new net LEFT: U4.4
- new net ON: R19.2
- new net RIGHT: U4.2
- new net SLEEP_MODE: R20.2
- new net STOP: U4.6
- no-connect marks 0 -> 9
Other:
- note added: "UI Submodule"
- company: (none) -> PRES
- title: (none) -> UI Submodule

Commit message: converter values adjusted
Changed lines of the file:
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@@
-	)
-	(junction
-		(at 255.27 121.92)
-		(diameter 0)
-		(color 0 0 0 0)
 	)
 	(junction
@@
 	(wire
 		(pts
-			(xy 261.62 121.92) (xy 255.27 121.92)
-		)
-		(stroke
-			(width 0)
-			(type default)
-		)
-	)
-	(wire
-		(pts
 			(xy 92.71 81.28) (xy 111.76 81.28)
 		)
@@
 			(font
 				(size 1.27 1.27)
-				(thickness 0.254)
-				(bold yes)
+				(thickness 0.1588)
 			)
 			(justify left)
@@
 			(font
 				(size 1.27 1.27)
-				(thickness 0.254)
-				(bold yes)
+				(thickness 0.1588)
 			)
 			(justify left)
@@
 			(font
 				(size 1.27 1.27)
-				(thickness 0.254)
-				(bold yes)
+				(thickness 0.1588)
 			)
 			(justify left)
